File: Circuit/communication_body/communication_body.kicad_pcb (KiCad board)
At the start: 2 copper layers, 50 x 55 mm, 44 parts, among them J1 SPI, J2 UART, J4 Power, J5 Control, J6 Camera, J7 USB, SW1 Reset, U1 RFM95W-868S2, U2 CH340G, U3 ATmega328P-A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

Commit message: Add Ground control circuit, Modify the rest and add payment confirmation details from manufacture
Parts:
- J7: footprint Connector_USB:USB_Micro-B_Molex_47346-0001 -> Connector_USB:USB_Micro-B_Amphenol_10118194_Horizontal
Changed lines of the file:
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@@
 		(allow_soldermask_bridges_in_footprints no)
 		(pcbplotparams
-			(layerselection 0x00010ff_ffffffff)
+			(layerselection 0x003ffff_ffffffff)
 			(plot_on_all_layers_selection 0x0000000_00000000)
 			(disableapertmacros no)
@@
 			(drillshape 0)
 			(scaleselection 1)
-			(outputdirectory "Drills/")
+			(outputdirectory "Gerbers/")
 		)
 	)
@@
 		(sheetname "Root")
 		(sheetfile "communication_body.kicad_sch")
-		(attr exclude_from_pos_files)
+		(attr exclude_from_pos_files exclude_from_bom)
 		(fp_circle
 			(center 0 0)
@@
 		(sheetname "Root")
 		(sheetfile "communication_body.kicad_sch")
-		(attr exclude_from_pos_files)
+		(attr exclude_from_pos_files exclude_from_bom)
 		(fp_circle
 			(center 0 0)
@@
 		)
 	)
-	(footprint "Connector_USB:USB_Micro-B_Molex_47346-0001"
+	(footprint "Connector_USB:USB_Micro-B_Amphenol_10118194_Horizontal"
 		(layer "F.Cu")
 		(at 115.39 116.8525 -90)
-		(descr "Micro USB B receptable with flange, bottom-mount, SMD, right-angle (http://www.molex.com/pdm_docs/sd/473460001_sd.pdf)")
-		(tags "Micro B USB SMD")
+		(descr "USB Micro-B receptacle, horizontal, SMD, 10118194, https://cdn.amphenol-icc.com/media/wysiwyg/files/drawing/10118194.pdf")
+		(tags "USB Micro B horizontal SMD")
 		(property "Reference" "J7"
-			(at -0.5975 -3.475 90)
+			(at 0 -3.5 -90)
 			(layer "F.SilkS")
 			(effects
@@
 		)
 		(property "Value" "USB"
-			(at 2.3525 -3.265 90)
+			(at 0 4.75 -90)
 			(layer "F.Fab")
 			(effects
@@
 			)
 		)
-		(property "Footprint" "Connector_USB:USB_Micro-B_Molex_47346-0001"
+		(property "Footprint" "Connector_USB:USB_Micro-B_Amphenol_10118194_Horizontal"
 			(at 0 0 -90)
 			(unlocked yes)
@@
 		(attr smd)
 		(fp_line
-			(start -3.81 2.6)
-			(end -3.81 2.34)
+			(start -3.76 2.69)
+			(end -3.76 2.29)
+			(stroke
+				(width 0.12)
+				(type solid)
+			)
+			(layer "F.SilkS")
+		)
+		(fp_line
+			(start 3.76 2.29)
+			(end 3.76 2.69)
 			(stroke
 				(width 0.12)
@@
 		)
 		(fp_line
-			(start 3.81 2.34)
-			(end 3.81 2.6)
+			(start -3.76 0.32)
+			(end -3.76 -1.66)
 			(stroke
 				(width 0.12)
@@
 		)
 		(fp_line
-			(start -3.81 0.06)
-			(end -3.81 -1.71)
+			(start 3.76 0.32)
+			(end 3.76 -1.66)
 			(stroke
 				(width 0.12)
@@
 		)
 		(fp_line
-			(start -3.81 -1.71)
-			(end -3.43 -1.71)
+			(start -3.76 -1.66)
+			(end -3.34 -1.66)
 			(stroke
 				(width 0.12)
@@
 		)
 		(fp_line
-			(start 3.81 -1.71)
-			(end 3.81 0.06)
+			(start 3.76 -1.66)
+			(end 3.34 -1.66)
 			(stroke
 				(width 0.12)
@@
 		)
 		(fp_line
-			(start 3.81 -1.71)
-			(end 3.43 -1.71)
+			(start -1.76 -1.89)
+			(end -1.76 -2.34)
 			(stroke
 				(width 0.12)
@@
 		)
 		(fp_line
-			(start -4.7 3.85)
-			(end -4.7 -2.65)
+			(start -1.31 -2.34)
+			(end -1.76 -2.34)
+			(stroke
+				(width 0.12)
+				(type solid)
+			)
+			(layer "F.SilkS")
+		)
+		(fp_line
+			(start 3 2.75)
+			(end -3 2.75)
+			(stroke
+				(width 0.1)
+				(type solid)
+			)
+			(layer "Dwgs.User")
+		)
+		(fp_line
+			(start -4.45 3.95)
+			(end 4.45 3.95)
 			(stroke
 				(width 0.05)
@@
 		)
 		(fp_line
-			(start 4.7 3.85)
-			(end -4.7 3.85)
+			(start -4.45 -2.58)
+			(end -4.45 3.95)
 			(stroke
 				(width 0.05)
@@
 		)
 		(fp_line
-			(start -4.7 -2.65)
-			(end 4.7 -2.65)
+			(start -4.45 -2.58)
+			(end 4.45 -2.58)
 			(stroke
 				(width 0.05)
@@
 		)
 		(fp_line
-			(start 4.7 -2.65)
-			(end 4.7 3.85)
+			(start 4.45 -2.58)
+			(end 4.45 3.95)
 			(stroke
 				(width 0.05)
@@
 		)
 		(fp_line
-			(start -3.75 3.35)
-			(end -3.75 -1.65)
+			(start -3.65 3.45)
+			(end -3.65 -0.55)
 			(stroke
 				(width 0.1)
@@
 		)
 		(fp_line
-			(start 3.75 3.35)
-			(end -3.75 3.35)
+			(start 3.65 3.45)
+			(end -3.65 3.45)
 			(stroke
 				(width 0.1)
@@
 		)
 		(fp_line
-			(start -3.25 2.65)
-			(end 3.25 2.65)
+			(start -3.65 -0.55)
+			(end -2.65 -1.55)
 			(stroke
 				(width 0.1)
@@
 		)
 		(fp_line
-			(start -3.75 -1.65)
-			(end 3.75 -1.65)
+			(start -2.65 -1.55)
+			(end 3.65 -1.55)
 			(stroke
 				(width 0.1)
@@
 		)
 		(fp_line
-			(start 3.75 -1.65)
-			(end 3.75 3.35)
+			(start 3.65 -1.55)
+			(end 3.65 3.45)
 			(stroke
 				(width 0.1)
@@
 		)
 		(fp_text user "PCB Edge"
-			(at 0 2.67 90)
+			(at 0 2.75 -90)
 			(layer "Dwgs.User")
 			(effects
 				(font
-					(size 0.4 0.4)
-					(thickness 0.04)
+					(size 0.5 0.5)
+					(thickness 0.08)
 				)
 			)
 		)
 		(fp_text user "${REFERENCE}"
-			(at 0 1.2 90)
+			(at 0 -0.05 -90)
 			(layer "F.Fab")
 			(effects
@@
 			)
 		)
+		(pad "" smd oval
+			(at -3.5 1.3 270)
+			(size 0.89 1.55)
+			(layers "F.Paste")
+		)
+		(pad "" smd oval
+			(at -2.5 -1.4 270)
+			(size 1.25 0.95)
+			(layers "F.Paste")
+		)
+		(pad "" smd oval
+			(at 2.5 -1.4 270)
+			(size 1.25 0.95)
+			(layers "F.Paste")
+		)
+		(pad "" smd oval
+			(at 3.5 1.3 270)
+			(size 0.89 1.55)
+			(layers "F.Paste")
+		)
 		(pad "1" smd rect
-			(at -1.3 -1.46 270)
-			(size 0.45 1.38)
+			(at -1.3 -1.4 270)
+			(size 0.4 1.35)
 			(layers "F.Cu" "F.Paste" "F.Mask")
 			(net 43 "Net-(D4-A)")
@@
 		)
 		(pad "2" smd rect
-			(at -0.65 -1.46 270)
-			(size 0.45 1.38)
+			(at -0.65 -1.4 270)
+			(size 0.4 1.35)
 			(layers "F.Cu" "F.Paste" "F.Mask")
 			(net 45 "Net-(J7-D-)")
@@
 		)
 		(pad "3" smd rect
-			(at 0 -1.46 270)
-			(size 0.45 1.38)
+			(at 0 -1.4 270)
+			(size 0.4 1.35)
 			(layers "F.Cu" "F.Paste" "F.Mask")
 			(net 46 "Net-(J7-D+)")
@@
 		)
 		(pad "4" smd rect
-			(at 0.65 -1.46 270)
-			(size 0.45 1.38)
+			(at 0.65 -1.4 270)
+			(size 0.4 1.35)
 			(layers "F.Cu" "F.Paste" "F.Mask")
 			(net 44 "unconnected-(J7-ID-Pad4)")
@@
 		)
 		(pad "5" smd rect
-			(at 1.3 -1.46 270)
-			(size 0.45 1.38)
+			(at 1.3 -1.4 270)
+			(size 0.4 1.35)
 			(layers "F.Cu" "F.Paste" "F.Mask")
 			(net 1 "GND")
@@
 			(pintype "power_out")
 		)
-		(pad "6" smd rect
-			(at -3.375 1.2 270)
-			(size 1.65 1.3)
-			(layers "F.Cu" "F.Paste" "F.Mask")
+		(pad "6" thru_hole oval
+			(at -3.5 1.3 270)
+			(size 0.89 1.55)
+			(drill oval 0.5 1.15)
+			(layers "*.Cu" "*.Mask")
+			(remove_unused_layers no)
 			(net 1 "GND")
 			(pinfunction "Shield")
@@
 		)
 		(pad "6" smd rect
-			(at -2.4875 -1.375 270)
-			(size 1.425 1.55)
+			(at -2.9 1.3 270)
+			(size 1.2 1.55)
 			(layers "F.Cu" "F.Paste" "F.Mask")
 			(net 1 "GND")
@@
 			(pintype "passive")
 		)
-		(pad "6" smd rect
-			(at -1.15 1.2 270)
-			(size 1.8 1.9)
-			(layers "F.Cu" "F.Paste" "F.Mask")
+		(pad "6" thru_hole oval
+			(at -2.5 -1.4 270)
+			(size 1.25 0.95)
+			(drill oval 0.85 0.55)
+			(layers "*.Cu" "*.Mask")
+			(remove_unused_layers no)
 			(net 1 "GND")
 			(pinfunction "Shield")
@@
 		)
 		(pad "6" smd rect
-			(at 1.55 1.2 270)
-			(size 1 1.9)
+			(at -1 1.3 270)
+			(size 1.5 1.55)
 			(layers "F.Cu" "F.Paste" "F.Mask")
 			(net 1 "GND")
@@
 		)
 		(pad "6" smd rect
-			(at 2.4875 -1.375 270)
-			(size 1.425 1.55)
+			(at 1 1.3 270)
+			(size 1.5 1.55)
 			(layers "F.Cu" "F.Paste" "F.Mask")
 			(net 1 "GND")
@@
 			(pintype "passive")
 		)
+		(pad "6" thru_hole oval
+			(at 2.5 -1.4 270)
+			(size 1.25 0.95)
+			(drill oval 0.85 0.55)
+			(layers "*.Cu" "*.Mask")
+			(remove_unused_layers no)
+			(net 1 "GND")
+			(pinfunction "Shield")
+			(pintype "passive")
+		)
 		(pad "6" smd rect
-			(at 3.375 1.2 270)
-			(size 1.65 1.3)
+			(at 2.9 1.3 270)
+			(size 1.2 1.55)
 			(layers "F.Cu" "F.Paste" "F.Mask")
 			(net 1 "GND")
@@
 			(pintype "passive")
 		)
-		(model "${KICAD8_3DMODEL_DIR}/Connector_USB.3dshapes/USB_Micro-B_Molex_47346-0001.wrl"
+		(pad "6" thru_hole oval
+			(at 3.5 1.3 270)
+			(size 0.89 1.55)
+			(drill oval 0.5 1.15)
+			(layers "*.Cu" "*.Mask")
+			(remove_unused_layers no)
+			(net 1 "GND")
+			(pinfunction "Shield")
+			(pintype "passive")
+		)
+		(model "${KICAD8_3DMODEL_DIR}/Connector_USB.3dshapes/USB_Micro-B_Amphenol_10118194_Horizontal.wrl"
 			(offset
 				(xyz 0 0 0)
@@
 		(sheetname "Root")
 		(sheetfile "communication_body.kicad_sch")
-		(attr exclude_from_pos_files)
+		(attr exclude_from_pos_files exclude_from_bom)
 		(fp_circle
 			(center 0 0)
