File: Circuit/communication_body/communication_body.kicad_sch (KiCad schematic)
At the start: 44 parts, among them J1 SPI, J2 UART, J4 Power, J5 Control, J6 Camera, J7 USB, SW1 Reset, U1 RFM95W-868S2, U2 CH340G, U3 ATmega328P-A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

Commit message: Add Ground control circuit, Modify the rest and add payment confirmation details from manufacture
Parts:
- J7: footprint Connector_USB:USB_Micro-B_Molex_47346-0001 -> Connector_USB:USB_Micro-B_Amphenol_10118194_Horizontal
Changed lines of the file:
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@@
 			)
 		)
-		(property "Footprint" "Connector_USB:USB_Micro-B_Molex_47346-0001"
+		(property "Footprint" "Connector_USB:USB_Micro-B_Amphenol_10118194_Horizontal"
 			(at 31.75 166.37 0)
 			(effects
