File: Circuit/control_body/control_body.kicad_pcb (KiCad board)
At the start: 2 copper layers, 80 x 65 mm, 111 parts, among them J1 Servo, J10 Proximity, J11 Servo, J12 Servo, J13 Servo, J14 POWER, J15 Proximity, J16 Proximity, J17 Proximity, J18 Proximity, J19 Proximity, J2 USB, J20 Communication, J21 SPI, J23 Lights connectors, J3 SPI, J4 UART, J5 ESC, J6 ESC, J7 ESC, J8 ESC, J9 ESC, Q1 IRF7380, Q2 IRF7380, Q3 IRF7380, Q4 IRF540NS, Q5 UMH3N, Q6 UMH3N, Q7 UMH3N, Q9 PZT2222A, SW1 Reset BTN, SW2 BTN1, SW3 BTN2, U1 CH340G, U2 ATmega2561-16A, U3 SIM28ML, U4 BMP280, U5 MPU-9150, U6 NE555D, U7 ATtiny85-20S, Y1 12MHz, Y2 16MHz

Commit message: Add Ground control circuit, Modify the rest and add payment confirmation details from manufacture
Parts:
- C16: value 22pF -> 10uF
- J2: footprint Connector_USB:USB_Micro-B_Molex_47346-0001 -> Connector_USB:USB_Micro-B_Amphenol_10118194_Horizontal
- R1: value R -> 6.2k
- R19: value 10k -> 72k
- R3: value R -> 47k
- R4: value R -> 4.7k
Connections:
- AE1 pad 2: GND -> +5V
- AE2 pad 2: GND -> +5V
- BZ1 pad 2: GND -> +5V
- C1 pad 2: GND -> +5V
- C10 pad 2: GND -> +5V
- C11 pad 1: GND -> +5V
- C12 pad 1: GND -> +5V
- C13 pad 1: GND -> +5V
- C14 pad 1: GND -> +5V
- C15 pad 1: GND -> +5V
- C16 pad 1: GND -> +5V
- C2 pad 1: GND -> +5V
- C3 pad 1: GND -> +5V
- C4 pad 1: GND -> +5V
- C5 pad 1: GND -> +5V
- C6 pad 2: GND -> +5V
- C7 pad 1: GND -> +5V
- C8 pad 1: GND -> +5V
- C9 pad 1: GND -> +5V
- D2 pad 1: GND -> +5V
- D3 pad 1: GND -> +5V
- D4 pad 2: GND -> +5V
- D6 pad 1: GND -> +5V
- H1 pad 1: GND -> +5V
- H2 pad 1: GND -> +5V
- H3 pad 1: GND -> +5V
- H4 pad 1: GND -> +5V
- J1 pad 3: GND -> +5V
- J10 pad 3: GND -> +5V
- J11 pad 3: GND -> +5V
- J12 pad 3: GND -> +5V
- J13 pad 3: GND -> +5V
- J14 pad 5: GND -> +5V
- J15 pad 3: GND -> +5V
- J16 pad 3: GND -> +5V
- J17 pad 3: GND -> +5V
- J18 pad 3: GND -> +5V
- J19 pad 3: GND -> +5V
- J2 pad 5: GND -> +5V
- J2 pad 6: GND -> +5V
- J20 pad 1: GND -> +5V
- J21 pad 4: GND -> +5V
- J23 pad 12: GND -> +5V
- J3 pad 4: GND -> +5V
- J4 pad 4: GND -> +5V
- J5 pad 3: GND -> +5V
- J6 pad 3: GND -> +5V
- J7 pad 3: GND -> +5V
- J8 pad 3: GND -> +5V
- J9 pad 3: GND -> +5V
- JP1 pad 1: GND -> +5V
- JP2 pad 3: GND -> +5V
- JP3 pad 1: GND -> +5V
- Q1 pad 1: GND -> +5V
- Q1 pad 3: GND -> +5V
- Q2 pad 1: GND -> +5V
- Q2 pad 3: GND -> +5V
- Q3 pad 1: GND -> +5V
- Q3 pad 3: GND -> +5V
- Q4 pad 3: GND -> +5V
- Q5 pad 1: GND -> +5V
- Q5 pad 4: GND -> +5V
- Q6 pad 1: GND -> +5V
- Q6 pad 4: GND -> +5V
- Q7 pad 1: GND -> +5V
- Q7 pad 4: GND -> +5V
- Q9 pad 3: GND -> +5V
- R4 pad 2: GND -> +5V
- SW1 pad 1: GND -> +5V
- SW2 pad 2: GND -> +5V
- SW3 pad 2: GND -> +5V
- U1 pad 1: GND -> +5V
- U2 pad 22: GND -> +5V
- U2 pad 53: GND -> +5V
- U2 pad 63: GND -> +5V
- U3 pad 1: GND -> +5V
- U3 pad 10: GND -> +5V
- U3 pad 12: GND -> +5V
- U4 pad 1: GND -> +5V
- U4 pad 5: GND -> +5V
- U4 pad 7: GND -> +5V
- U5 pad 15: GND -> +5V
- U5 pad 17: GND -> +5V
- U5 pad 18: GND -> +5V
- U6 pad 1: GND -> +5V
- U7 pad 4: GND -> +5V
Routing:
- net +5V: track 336.7 -> 364.3 mm, vias 10 -> 124
- net GND: track 27.6 -> 0.00 mm, vias 114 -> 0
- added copper zone on B.Cu, net +5V
- added copper zone on F.Cu, net +5V
- removed copper zone on B.Cu, net GND
- removed copper zone on F.Cu, net GND
