File: Circuit/control_body/control_unit.kicad_sch (KiCad schematic)
At the start: 53 parts, among them J1 Servo, J11 Servo, J12 Servo, J13 Servo, J14 POWER, J2 USB, J20 Communication, J3 SPI, J4 UART, J5 ESC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

Commit message: Add Ground control circuit, Modify the rest and add payment confirmation details from manufacture
Parts:
- J2: footprint Connector_USB:USB_Micro-B_Molex_47346-0001 -> Connector_USB:USB_Micro-B_Amphenol_10118194_Horizontal
Changed lines of the file:
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@@
 			)
 		)
-		(property "Footprint" "Connector_USB:USB_Micro-B_Molex_47346-0001"
+		(property "Footprint" "Connector_USB:USB_Micro-B_Amphenol_10118194_Horizontal"
 			(at 43.18 68.58 0)
 			(effects
